File: Ganglion_KiCad_Files/Ganglion_01.sch (KiCad schematic (older format))
At the start: 86 parts, among them P1 CONN_02X10, P2 CONN_01X04, P3 CONN_01X04, P4 CONN_01X08, P5 CONN_01X08, SW1 CJS1200, SW2 CJS1200, SW3 CJS1200, SW4 CJS1200, SW5 SPDT, SW6 TACT_SWITCH, U10 NCP300, U11 NCP551, U2 AD8237, U3 AD8237, U4 AD8237, U5 AD8237, U6 LM7332, U7 MCP3912, U8 rfd_77101, U9 NCP551, Y1 Xtal

Commit message: added PDF of Schematic
Parts:
- added C?: 1uF, Capacitors_SMD:C_0603, symbol C
- added R? (x2): 100K, Resistors_SMD:R_0603, symbol R
- added U?: MCP6V31U, symbol MCP6V31U
Connections:
- net labels added: DRIVEN_GND
- wire segments 389 -> 404
Other:
- moved on the sheet: C14
Changed lines of the file:
@@
 Connection ~ 2350 8300
 Wire Wire Line
-	2550 8700 3300 8700
+	2550 8700 3200 8700
 Wire Wire Line
 	2550 8900 2600 8900
@@
 L C C14
 U 1 1 5722FC73
-P 3300 8950
-F 0 "C14" H 3300 8850 50  0000 L CNN
-F 1 "1uF" H 3300 9050 50  0000 L CNN
-F 2 "Capacitors_SMD:C_0603" H 3338 8800 50  0001 C CNN
-F 3 "" H 3300 8950 50  0000 C CNN
-	1    3300 8950
-	1    0    0    -1
-$EndComp
-Wire Wire Line
-	3300 8700 3300 8800
-Wire Wire Line
-	3300 9250 3300 9100
+P 3200 8950
+F 0 "C14" H 3200 8850 50  0000 L CNN
+F 1 "1uF" H 3200 9050 50  0000 L CNN
+F 2 "Capacitors_SMD:C_0603" H 3238 8800 50  0001 C CNN
+F 3 "" H 3200 8950 50  0000 C CNN
+	1    3200 8950
+	1    0    0    -1
+$EndComp
+Wire Wire Line
+	3200 8700 3200 8800
+Wire Wire Line
+	3200 9250 3200 9100
 Wire Wire Line
 	1800 1700 1800 2200
@@
 pull down here!
 Wire Wire Line
-	2350 9250 3300 9250
+	2350 9250 3200 9250
 $Comp
 L JS_2_Battery B1
@@
 S 5650 5500 1150 400
 U 57E20C3A
-F0 "Ganglion_V_REF" 60
+F0 "INPUT_V_REF" 60
 F1 "References.sch" 60
 $EndSheet
@@
 	5850 4250 5650 4250
 Connection ~ 5650 4250
+$Comp
+L MCP6V31U U?
+U 1 1 580687F8
+P 5050 8800
+F 0 "U?" H 5100 9000 50  0000 C CNN
+F 1 "MCP6V31U" H 5250 8600 50  0000 C CNN
+F 2 "" H 5000 8900 50  0000 C CNN
+F 3 "" H 5100 9000 50  0000 C CNN
+	1    5050 8800
+	-1   0    0    -1
+$EndComp
+$Comp
+L R R?
+U 1 1 58068B01
+P 5700 8500
+F 0 "R?" V 5780 8500 50  0000 C CNN
+F 1 "100K" V 5700 8500 50  0000 C CNN
+F 2 "Resistors_SMD:R_0603" V 5630 8500 50  0001 C CNN
+F 3 "" H 5700 8500 50  0000 C CNN
+	1    5700 8500
+	1    0    0    -1
+$EndComp
+$Comp
+L R R?
+U 1 1 58068C34
+P 5700 8900
+F 0 "R?" V 5780 8900 50  0000 C CNN
+F 1 "100K" V 5700 8900 50  0000 C CNN
+F 2 "Resistors_SMD:R_0603" V 5630 8900 50  0001 C CNN
+F 3 "" H 5700 8900 50  0000 C CNN
+	1    5700 8900
+	1    0    0    -1
+$EndComp
+$Comp
+L C C?
+U 1 1 5806964A
+P 5950 8900
+F 0 "C?" H 5950 8800 50  0000 L CNN
+F 1 "1uF" H 5950 9000 50  0000 L CNN
+F 2 "Capacitors_SMD:C_0603" H 5988 8750 50  0001 C CNN
+F 3 "" H 5950 8900 50  0000 C CNN
+	1    5950 8900
+	1    0    0    -1
+$EndComp
+$Comp
+L VAA #PWR?
+U 1 1 58069B6B
+P 5150 8250
+F 0 "#PWR?" H 5150 8100 50  0001 C CNN
+F 1 "VAA" H 5150 8400 50  0000 C CNN
+F 2 "" H 5150 8250 50  0000 C CNN
+F 3 "" H 5150 8250 50  0000 C CNN
+	1    5150 8250
+	1    0    0    -1
+$EndComp
+$Comp
+L GNDA #PWR?
+U 1 1 58069C87
+P 5150 9300
+F 0 "#PWR?" H 5150 9050 50  0001 C CNN
+F 1 "GNDA" H 5150 9150 50  0000 C CNN
+F 2 "" H 5150 9300 50  0000 C CNN
+F 3 "" H 5150 9300 50  0000 C CNN
+	1    5150 9300
+	1    0    0    -1
+$EndComp
+Wire Wire Line
+	5150 8250 5150 8500
+Wire Wire Line
+	5700 8350 5700 8300
+Wire Wire Line
+	5700 8300 5150 8300
+Connection ~ 5150 8300
+Wire Wire Line
+	5150 9100 5150 9300
+Wire Wire Line
+	5700 9050 5700 9250
+Wire Wire Line
+	5150 9250 5950 9250
+Connection ~ 5150 9250
+Wire Wire Line
+	5350 8900 5450 8900
+Wire Wire Line
+	5450 8900 5450 9150
+Wire Wire Line
+	5450 9150 4550 9150
+Wire Wire Line
+	4550 9150 4550 8800
+Wire Wire Line
+	4550 8800 4750 8800
+Wire Wire Line
+	5350 8700 5950 8700
+Wire Wire Line
+	5700 8650 5700 8750
+Connection ~ 5700 8700
+Wire Wire Line
+	5950 8700 5950 8750
+Wire Wire Line
+	5950 9250 5950 9050
+Connection ~ 5700 9250
+Text GLabel 4550 8800 0    60   Input ~ 0
+DRIVEN_GND
 $EndSCHEMATC

Commit message: small changes
improved readability of shcematic
Connections:
- net labels added: D_G
- net labels removed: DRIVEN_GND, DRL, GUARD
Other:
- note added: "DRIVEN GROUND"
- note added: "INPUT CURRENT BIAS"
- moved on the sheet: C16, C17, C22, C23, D2, P2, P3, P4, P5, R47

Commit message: small changes
Parts:
- removed P1: CONN_02X10, Pin_Headers:Pin_Header_Angled_2x10, symbol CONN_02X10
- added P1: CONN_02X08, Pin_Headers:Pin_Header_Angled_2x08, symbol CONN_02X08
- U25: renamed from U?; footprint (none) -> TO_SOT_Packages_SMD:SC-70-5
- gave numbers to parts that had none: 3
Connections:
- net labels added: REF+_OUT
- wire segments 404 -> 416
Other:
- note added: "INPUT HEADER"
- moved on the sheet: D2, P2, P3, P4, P5, R47

Commit message: Commit PCB files
Update with the production schematic and PCB files. Also  the BOM.
You’re welcome.
Parts:
- removed Y1: Xtal, OpenBCI:ABM3C, symbol Xtal
- added C46: 1uF, Capacitors_SMD:C_0603, symbol C
- added R49: 330K, Resistors_SMD:R_0603, symbol R
- added Y1: Crystal_Small, Crystals:Crystal_HC49-SD_SMD, symbol Crystal_Small
Other:
- note added: "ABLS-LR-3.2768MHZ-T\n"
- note removed: "ABM3C-19.6608MHZ-D4Y-T"
- moved on the sheet: C43, C45, R32, R33, U25
Changed lines of the file:
@@
 F 3 "" H 11550 2800 50  0000 C CNN
 	1    11550 2800
-	1    0    0    -1
+	1    0    0    1
 $EndComp
 $Comp
@@
 Wire Wire Line
 	10650 2700 10650 2550
-Wire Wire Line
-	11250 2550 11250 2800
-Wire Wire Line
-	11850 2700 11950 2700
-Wire Wire Line
-	11950 2700 11950 2550
-Connection ~ 11250 2550
 Wire Wire Line
 	11850 2900 13000 2900
@@
 Wire Wire Line
 	10650 2550 10800 2550
-Wire Wire Line
-	11950 2550 11100 2550
 $Comp
 L TACT_SWITCH SW6
@@
 L C C43
 U 1 1 57437A41
-P 8050 2900
-F 0 "C43" H 7900 3000 50  0000 L CNN
-F 1 "18pF" H 7850 2800 50  0000 L CNN
-F 2 "Capacitors_SMD:C_0603" H 8088 2750 50  0001 C CNN
-F 3 "" H 8050 2900 50  0000 C CNN
-	1    8050 2900
+P 8050 2850
+F 0 "C43" H 7900 2950 50  0000 L CNN
+F 1 "18pF" H 7850 2750 50  0000 L CNN
+F 2 "Capacitors_SMD:C_0603" H 8088 2700 50  0001 C CNN
+F 3 "" H 8050 2850 50  0000 C CNN
+	1    8050 2850
 	-1   0    0    1
 $EndComp
 Wire Wire Line
-	8050 3050 8050 3100
+	8050 3000 8050 3100
 Connection ~ 8050 3100
 Wire Wire Line
-	8050 2400 8050 2750
+	8050 2400 8050 2700
 $Comp
 L LED D2
@@
 Wire Wire Line
 	8050 2400 7200 2400
-Connection ~ 8050 2700
-$Comp
-L Xtal Y1
-U 1 1 57E198AB
-P 8500 2500
-F 0 "Y1" V 8500 2500 50  0000 C CNN
-F 1 "Xtal" V 8450 2700 50  0000 C CNN
-F 2 "OpenBCI:ABM3C" H 8500 2500 50  0001 C CNN
-F 3 "" H 8500 2500 50  0000 C CNN
-	1    8500 2500
-	0    1    1    0
-$EndComp
-Wire Wire Line
-	8700 2500 8700 3100
-Connection ~ 8700 3100
-Wire Wire Line
-	8300 2500 8300 3100
-Connection ~ 8300 3100
-Text Notes 7900 3250 0    60   ~ 0
-ABM3C-19.6608MHZ-D4Y-T
+Text Notes 8000 3250 0    60   ~ 0
+ABLS-LR-3.2768MHZ-T\n
 Wire Wire Line
 	7200 2300 8950 2300
-Wire Wire Line
-	8500 2350 8500 2300
-Connection ~ 8500 2300
-Wire Wire Line
-	8500 2650 8500 2700
-Wire Wire Line
-	8500 2700 8050 2700
 $Comp
 L C C38
@@
 L MCP6V31U U25
 U 1 1 580687F8
-P 5050 8800
-F 0 "U25" H 5100 9000 50  0000 C CNN
-F 1 "MCP6V31U" H 5250 8600 50  0000 C CNN
-F 2 "TO_SOT_Packages_SMD:SC-70-5" H 5000 8900 50  0001 C CNN
-F 3 "" H 5100 9000 50  0000 C CNN
-	1    5050 8800
+P 5550 8800
+F 0 "U25" H 5600 9000 50  0000 C CNN
+F 1 "MCP6V31U" H 5750 8600 50  0000 C CNN
+F 2 "TO_SOT_Packages_SMD:SC-70-5" H 5500 8900 50  0001 C CNN
+F 3 "" H 5600 9000 50  0000 C CNN
+	1    5550 8800
 	-1   0    0    -1
 $EndComp
@@
 L R R32
 U 1 1 58068B01
-P 5700 8500
-F 0 "R32" V 5780 8500 50  0000 C CNN
-F 1 "100K" V 5700 8500 50  0000 C CNN
-F 2 "Resistors_SMD:R_0603" V 5630 8500 50  0001 C CNN
-F 3 "" H 5700 8500 50  0000 C CNN
-	1    5700 8500
+P 6200 8500
+F 0 "R32" V 6280 8500 50  0000 C CNN
+F 1 "100K" V 6200 8500 50  0000 C CNN
+F 2 "Resistors_SMD:R_0603" V 6130 8500 50  0001 C CNN
+F 3 "" H 6200 8500 50  0000 C CNN
+	1    6200 8500
 	1    0    0    -1
 $EndComp
@@
 L R R33
 U 1 1 58068C34
-P 5700 8900
-F 0 "R33" V 5780 8900 50  0000 C CNN
-F 1 "100K" V 5700 8900 50  0000 C CNN
-F 2 "Resistors_SMD:R_0603" V 5630 8900 50  0001 C CNN
-F 3 "" H 5700 8900 50  0000 C CNN
-	1    5700 8900
+P 6200 8900
+F 0 "R33" V 6280 8900 50  0000 C CNN
+F 1 "100K" V 6200 8900 50  0000 C CNN
+F 2 "Resistors_SMD:R_0603" V 6130 8900 50  0001 C CNN
+F 3 "" H 6200 8900 50  0000 C CNN
+	1    6200 8900
 	1    0    0    -1
 $EndComp
@@
 L C C45
 U 1 1 5806964A
-P 5950 8900
-F 0 "C45" H 5950 8800 50  0000 L CNN
-F 1 "1uF" H 5950 9000 50  0000 L CNN
-F 2 "Capacitors_SMD:C_0603" H 5988 8750 50  0001 C CNN
-F 3 "" H 5950 8900 50  0000 C CNN
-	1    5950 8900
+P 6450 8900
+F 0 "C45" H 6450 8800 50  0000 L CNN
+F 1 "1uF" H 6450 9000 50  0000 L CNN
+F 2 "Capacitors_SMD:C_0603" H 6488 8750 50  0001 C CNN
+F 3 "" H 6450 8900 50  0000 C CNN
+	1    6450 8900
 	1    0    0    -1
 $EndComp
@@
 L VAA #PWR039
 U 1 1 58069B6B
-P 5150 8250
-F 0 "#PWR039" H 5150 8100 50  0001 C CNN
-F 1 "VAA" H 5150 8400 50  0000 C CNN
-F 2 "" H 5150 8250 50  0000 C CNN
-F 3 "" H 5150 8250 50  0000 C CNN
-	1    5150 8250
+P 5650 8250
+F 0 "#PWR039" H 5650 8100 50  0001 C CNN
+F 1 "VAA" H 5650 8400 50  0000 C CNN
+F 2 "" H 5650 8250 50  0000 C CNN
+F 3 "" H 5650 8250 50  0000 C CNN
+	1    5650 8250
 	1    0    0    -1
 $EndComp
@@
 L GNDA #PWR040
 U 1 1 58069C87
-P 5150 9300
-F 0 "#PWR040" H 5150 9050 50  0001 C CNN
-F 1 "GNDA" H 5150 9150 50  0000 C CNN
-F 2 "" H 5150 9300 50  0000 C CNN
-F 3 "" H 5150 9300 50  0000 C CNN
-	1    5150 9300
-	1    0    0    -1
-$EndComp
-Wire Wire Line
-	5150 8250 5150 8500
-Wire Wire Line
-	5700 8350 5700 8300
-Wire Wire Line
-	5700 8300 5150 8300
-Connection ~ 5150 8300
-Wire Wire Line
-	5150 9100 5150 9300
-Wire Wire Line
-	5700 9050 5700 9250
-Wire Wire Line
-	5150 9250 5950 9250
-Connection ~ 5150 9250
-Wire Wire Line
-	5350 8900 5450 8900
-Wire Wire Line
-	5450 8900 5450 9150
-Wire Wire Line
-	5450 9150 4550 9150
-Wire Wire Line
-	4550 9150 4550 8800
-Wire Wire Line
-	4400 8800 4750 8800
-Wire Wire Line
-	5350 8700 5950 8700
-Wire Wire Line
-	5700 8650 5700 8750
-Connection ~ 5700 8700
-Wire Wire Line
-	5950 8700 5950 8750
-Wire Wire Line
-	5950 9250 5950 9050
-Connection ~ 5700 9250
-Text Notes 4150 8650 0    60   ~ 0
+P 5650 9300
+F 0 "#PWR040" H 5650 9050 50  0001 C CNN
+F 1 "GNDA" H 5650 9150 50  0000 C CNN
+F 2 "" H 5650 9300 50  0000 C CNN
+F 3 "" H 5650 9300 50  0000 C CNN
+	1    5650 9300
+	1    0    0    -1
+$EndComp
+Wire Wire Line
+	5650 8250 5650 8500
+Wire Wire Line
+	6200 8350 6200 8300
+Wire Wire Line
+	6200 8300 5650 8300
+Connection ~ 5650 8300
+Wire Wire Line
+	5650 9100 5650 9300
+Wire Wire Line
+	6200 9050 6200 9250
+Wire Wire Line
+	5650 9250 6450 9250
+Connection ~ 5650 9250
+Wire Wire Line
+	5850 8900 5950 8900
+Wire Wire Line
+	5950 8900 5950 9150
+Wire Wire Line
+	5950 9150 4900 9150
+Wire Wire Line
+	5050 9150 5050 8800
+Wire Wire Line
+	4900 8800 5250 8800
+Wire Wire Line
+	5850 8700 6450 8700
+Wire Wire Line
+	6200 8650 6200 8750
+Connection ~ 6200 8700
+Wire Wire Line
+	6450 8700 6450 8750
+Wire Wire Line
+	6450 9250 6450 9050
+Connection ~ 6200 9250
+Text Notes 4650 8650 0    60   ~ 0
 DRIVEN GROUND
 Text Notes 1050 8700 0    60   ~ 0
 INPUT CURRENT BIAS
-Connection ~ 4550 8800
-Wire Wire Line
-	15400 6100 14350 6100
+Connection ~ 5050 8800
+Wire Wire Line
+	14350 6100 15400 6100
 Wire Wire Line
 	14600 6500 14600 6100
@@
 Text GLabel 4400 8800 0    60   Input ~ 0
 D_G
+$Comp
+L Crystal_Small Y1
+U 1 1 581B6085
+P 8500 2550
+F 0 "Y1" H 8500 2650 50  0000 C CNN
+F 1 "Crystal_Small" H 8500 2450 50  0000 C CNN
+F 2 "Crystals:Crystal_HC49-SD_SMD" H 8500 2550 50  0001 C CNN
+F 3 "" H 8500 2550 50  0000 C CNN
+	1    8500 2550
+	-1   0    0    1
+$EndComp
+Wire Wire Line
+	8600 2550 8950 2550
+Connection ~ 8950 2550
+Wire Wire Line
+	8400 2550 8050 2550
+Connection ~ 8050 2550
+Wire Wire Line
+	11950 2550 11950 2700
+Wire Wire Line
+	11950 2700 11850 2700
+Wire Wire Line
+	11250 2550 11250 2800
+Connection ~ 11250 2550
+Wire Wire Line
+	11100 2550 11950 2550
+$Comp
+L R R49
+U 1 1 581BB3E5
+P 4750 8800
+F 0 "R49" V 4830 8800 50  0000 C CNN
+F 1 "330K" V 4750 8800 50  0000 C CNN
+F 2 "Resistors_SMD:R_0603" V 4680 8800 50  0001 C CNN
+F 3 "" H 4750 8800 50  0000 C CNN
+	1    4750 8800
+	0    1    1    0
+$EndComp
+$Comp
+L C C46
+U 1 1 581BB528
+P 4750 9150
+F 0 "C46" H 4750 9050 50  0000 L CNN
+F 1 "1uF" H 4750 9250 50  0000 L CNN
+F 2 "Capacitors_SMD:C_0603" H 4788 9000 50  0001 C CNN
+F 3 "" H 4750 9150 50  0000 C CNN
+	1    4750 9150
+	0    1    1    0
+$EndComp
+Wire Wire Line
+	4400 8800 4600 8800
+Wire Wire Line
+	4600 9150 4500 9150
+Wire Wire Line
+	4500 9150 4500 8800
+Connection ~ 4500 8800
+Connection ~ 5050 9150
 $EndSCHEMATC
