File: Ganglion_KiCad_Files/Ganglion_01.sch (KiCad schematic (older format))
At the start: 92 parts, among them P1 CONN_02X08, P2 CONN_01X04, P3 CONN_01X04, P4 CONN_01X08, P5 CONN_01X08, SW1 CJS1200, SW2 CJS1200, SW3 CJS1200, SW4 CJS1200, SW5 SPDT, SW6 TACT_SWITCH, U10 NCP300, U11 NCP551, U2 AD8237, U25 MCP6V31U, U3 AD8237, U4 AD8237, U5 AD8237, U6 LM7332, U7 MCP3912, U8 rfd_77101, U9 NCP551, Y1 Crystal_Small

Commit message: Annotate components with manufacturer part numbers
Parts:
- B1: ManufacturerPartNumber (none) -> S2B-PH-SM4-TB(LF)(SN)
- C1, C15, C16, C2, C20, C21, C22, C24, C26, C27, C3, C31, C32, C4, C46, C5, C6, C7, C8: ManufacturerPartNumber (none) -> GRM188R71H104KA93D
- C10, C11, C12, C13, C14, C17, C19, C23, C25, C28, C30, C33, C45: ManufacturerPartNumber (none) -> GRM188R61E105KA12D
- C18, C29, C34: ManufacturerPartNumber (none) -> GRM188C80G106ME47D
- C38, C43: ManufacturerPartNumber (none) -> GRM1885C1H180JA01D
- D1: ManufacturerPartNumber (none) -> CDBU0130L
- D2: ManufacturerPartNumber (none) -> LTST-C193TBKT-5A
- P1: ManufacturerPartNumber (none) -> PRPC008DBAN-M71RC
- P2, P3: ManufacturerPartNumber (none) -> PPTC041LFBN-RC
- P4, P5: ManufacturerPartNumber (none) -> PPTC081LFBN-RC
- R11, R2, R3, R4, R49, R5, R6, R7, R8, R9: ManufacturerPartNumber (none) -> ERJ-3EKF3303V
- R15, R17, R19, R21, R27, R28, R32, R33, R37: ManufacturerPartNumber (none) -> ERJ-3EKF1003V
- R16, R18, R20, R22: ManufacturerPartNumber (none) -> ERJ-3EKF2001V
- R23, R24, R25, R26, R47: ManufacturerPartNumber (none) -> ERJ-3EKF1001V
- R38: ManufacturerPartNumber (none) -> ERJ-3EKF1002V
- SW1, SW2, SW3, SW4: ManufacturerPartNumber (none) -> CJS-1200TA
- SW5: ManufacturerPartNumber (none) -> SSSS810701
- SW6: ManufacturerPartNumber (none) -> PTS810 SJK 250 SMTR LFS
- U10: ManufacturerPartNumber (none) -> NCP300LSN30T1G
- U11, U9: ManufacturerPartNumber (none) -> NCP551SN30T1G
- U2, U3, U4, U5: ManufacturerPartNumber (none) -> AD8237ARMZ-R7
- U25: ManufacturerPartNumber (none) -> MCP6V31UT-E/LT
- U6: ManufacturerPartNumber (none) -> MCP6L02T-E/MS
- U7: ManufacturerPartNumber (none) -> MCP3912A1-E/SS
- U8: ManufacturerPartNumber (none) -> RFD77101
- Y1: ManufacturerPartNumber (none) -> ABLS-LR-3.2768MHZ-T
