File: Ganglion_KiCad_Files/Ganglion_Sensors_01.sch (KiCad schematic (older format))
At the start: 25 parts, among them U12 AD5621, U13 SEEED_microSD, U14 MCP6V13T, U15 MCP6001, U16 SN74LVC1G32, U17 LIS2DE12, U18 74LVC1G66, U19 74LVC1G66, U20 74LVC1G66, U21 74LVC1G66, U22 74LVC1G66, U23 74LVC2G00

Commit message: Commit PCB files
Update with the production schematic and PCB files. Also  the BOM.
You’re welcome.
Parts:
- U18, U19, U20, U21, U22: footprint TO_SOT_Packages_SMD:SOT-353 -> TO_SOT_Packages_SMD:SC-70-5
Changed lines of the file:
@@
 F 0 "U21" H 9900 4750 50  0000 C CNN
 F 1 "74LVC1G66" H 10000 4400 50  0000 C CNN
-F 2 "TO_SOT_Packages_SMD:SOT-353" H 9750 4600 60  0001 C CNN
+F 2 "TO_SOT_Packages_SMD:SC-70-5" H 9750 4600 60  0001 C CNN
 F 3 "" H 9750 4600 60  0000 C CNN
 	1    9750 4600
@@
 F 0 "U19" H 8850 3650 50  0000 C CNN
 F 1 "74LVC1G66" H 8950 3300 50  0000 C CNN
-F 2 "TO_SOT_Packages_SMD:SOT-353" H 8700 3500 60  0001 C CNN
+F 2 "TO_SOT_Packages_SMD:SC-70-5" H 8700 3500 60  0001 C CNN
 F 3 "" H 8700 3500 60  0000 C CNN
 	1    8700 3500
@@
 F 0 "U20" H 7850 4750 50  0000 C CNN
 F 1 "74LVC1G66" H 7950 4400 50  0000 C CNN
-F 2 "TO_SOT_Packages_SMD:SOT-353" H 7700 4600 60  0001 C CNN
+F 2 "TO_SOT_Packages_SMD:SC-70-5" H 7700 4600 60  0001 C CNN
 F 3 "" H 7700 4600 60  0000 C CNN
 	1    7700 4600
@@
 F 0 "U18" H 7850 5950 50  0000 C CNN
 F 1 "74LVC1G66" H 7950 5600 50  0000 C CNN
-F 2 "TO_SOT_Packages_SMD:SOT-353" H 7700 5800 60  0001 C CNN
+F 2 "TO_SOT_Packages_SMD:SC-70-5" H 7700 5800 60  0001 C CNN
 F 3 "" H 7700 5800 60  0000 C CNN
 	1    7700 5800
@@
 F 0 "U22" H 9900 5950 50  0000 C CNN
 F 1 "74LVC1G66" H 10000 5600 50  0000 C CNN
-F 2 "TO_SOT_Packages_SMD:SOT-353" H 9750 5800 60  0001 C CNN
+F 2 "TO_SOT_Packages_SMD:SC-70-5" H 9750 5800 60  0001 C CNN
 F 3 "" H 9750 5800 60  0000 C CNN
 	1    9750 5800
