File: Ganglion_KiCad_Files/References.sch (KiCad schematic (older format))
At the start: 16 parts, among them U1 MCP6V31U, U24 MCP6V31U, U25 MCP6V31T, U26 MCP6V31T

Commit message: added PDF of Schematic
Parts:
- removed U25, U26: MCP6V31T, TO_SOT_Packages_SMD:SOT-23-5, symbol MCP6001
- added R? (x4): 500K, Capacitors_SMD:C_0603, symbol R
- added U? (x2): MCP6V31U, symbol MCP6V31U
Connections:
- net GNDA: now also U1.5 (V+), U?.5 (V+), U?.5 (V+); no longer U1.2 (V-)
- net REF_2: now also U?.4
- net REF_4: now also U?.4
- net VAA: now also U1.2 (V-), U?.2 (V-), U?.2 (V-); no longer U1.5 (V+)
- net V_REF: now also R?.1, R?.1, R?.1, R?.1; no longer U1.3 (-), U24.3 (-)
- net at C9.1, R1.1, R12.2: now also U1.3 (-); no longer U1.1 (+)
- net at C37.1, R10.1, R13.2: now also U24.3 (-); no longer U24.1 (+)
- net at C44.1, R29.1: now also R?.2, U?.1 (+); no longer R31.2
- net at C39.1, R14.1, R30.2: now also U?.3 (-)
- new net: R31.2, U?.3 (-)
- new net: R?.2, U1.1 (+)
- new net: R?.2, U24.1 (+)
- new net: R?.2, U?.1 (+)
Other:
- moved on the sheet: R13, R30, R31
Changed lines of the file:
@@
 	0    1    1    0
 $EndComp
-Text GLabel 4550 2350 2    60   Input ~ 0
+Text GLabel 4950 2350 2    60   Input ~ 0
 V_REF
 $Comp
@@
 L R R13
 U 1 1 57EB8495
-P 7750 2350
-F 0 "R13" V 7830 2350 50  0000 C CNN
-F 1 "1M" V 7750 2350 50  0000 C CNN
-F 2 "Capacitors_SMD:C_0603" V 7680 2350 50  0001 C CNN
-F 3 "" H 7750 2350 50  0000 C CNN
-	1    7750 2350
+P 7750 2150
+F 0 "R13" V 7830 2150 50  0000 C CNN
+F 1 "1M" V 7750 2150 50  0000 C CNN
+F 2 "Capacitors_SMD:C_0603" V 7680 2150 50  0001 C CNN
+F 3 "" H 7750 2150 50  0000 C CNN
+	1    7750 2150
 	0    1    1    0
 $EndComp
@@
 $EndComp
 $Comp
-L MCP6001 U26
-U 1 1 57EB8511
-P 7000 4550
-F 0 "U26" H 7050 4750 50  0000 C CNN
-F 1 "MCP6V31T" H 7200 4350 50  0000 C CNN
-F 2 "TO_SOT_Packages_SMD:SOT-23-5" H 6950 4650 50  0001 C CNN
-F 3 "" H 7050 4750 50  0000 C CNN
-	1    7000 4550
-	-1   0    0    -1
-$EndComp
-$Comp
-L MCP6001 U25
-U 1 1 57EB854A
-P 4000 4550
-F 0 "U25" H 4050 4750 50  0000 C CNN
-F 1 "MCP6V31T" H 4200 4350 50  0000 C CNN
-F 2 "TO_SOT_Packages_SMD:SOT-23-5" H 3950 4650 50  0001 C CNN
-F 3 "" H 4050 4750 50  0000 C CNN
-	1    4000 4550
-	-1   0    0    -1
-$EndComp
-$Comp
 L C C39
 U 1 1 57EB85D4
@@
 L R R30
 U 1 1 57EB8682
-P 4700 4650
-F 0 "R30" V 4780 4650 50  0000 C CNN
-F 1 "1M" V 4700 4650 50  0000 C CNN
-F 2 "Capacitors_SMD:C_0603" V 4630 4650 50  0001 C CNN
-F 3 "" H 4700 4650 50  0000 C CNN
-	1    4700 4650
+P 4700 4450
+F 0 "R30" V 4780 4450 50  0000 C CNN
+F 1 "1M" V 4700 4450 50  0000 C CNN
+F 2 "Capacitors_SMD:C_0603" V 4630 4450 50  0001 C CNN
+F 3 "" H 4700 4450 50  0000 C CNN
+	1    4700 4450
 	0    1    1    0
 $EndComp
@@
 L R R31
 U 1 1 57EB86E1
-P 7700 4650
-F 0 "R31" V 7780 4650 50  0000 C CNN
-F 1 "1M" V 7700 4650 50  0000 C CNN
-F 2 "Capacitors_SMD:C_0603" V 7630 4650 50  0001 C CNN
-F 3 "" H 7700 4650 50  0000 C CNN
-	1    7700 4650
+P 7700 4450
+F 0 "R31" V 7780 4450 50  0000 C CNN
+F 1 "1M" V 7700 4450 50  0000 C CNN
+F 2 "Capacitors_SMD:C_0603" V 7630 4450 50  0001 C CNN
+F 3 "" H 7700 4450 50  0000 C CNN
+	1    7700 4450
 	0    1    1    0
 $EndComp
@@
 	1    0    0    -1
 $EndComp
-Text GLabel 4550 4450 2    60   Input ~ 0
+Text GLabel 4950 4650 2    60   Input ~ 0
 V_REF
-Text GLabel 7600 2150 2    60   Input ~ 0
+Text GLabel 8000 2350 2    60   Input ~ 0
 V_REF
-Text GLabel 7550 4450 2    60   Input ~ 0
+Text GLabel 8000 4650 2    60   Input ~ 0
 V_REF
 Wire Wire Line
@@
 	7100 2550 7100 2700
 Wire Wire Line
-	7300 2150 7600 2150
-Wire Wire Line
-	7300 4450 7550 4450
-Wire Wire Line
-	4300 4450 4550 4450
-Wire Wire Line
 	4000 3800 4450 3800
 Wire Wire Line
-	4450 3800 4450 4650
-Connection ~ 4450 4650
+	4450 3800 4450 4450
+Connection ~ 4450 4450
 Wire Wire Line
 	4000 4100 4450 4100
@@
 	7000 1500 7450 1500
 Wire Wire Line
-	7450 1500 7450 2350
-Connection ~ 7450 2350
+	7450 1500 7450 2150
+Connection ~ 7450 2150
 Wire Wire Line
 	7000 1800 7450 1800
@@
 Text GLabel 4950 2150 2    60   Input ~ 0
 OUT_1
-Text GLabel 4950 4650 2    60   Input ~ 0
+Text GLabel 4950 4450 2    60   Input ~ 0
 OUT_2
-Text GLabel 8000 2350 2    60   Input ~ 0
+Text GLabel 8000 2150 2    60   Input ~ 0
 OUT_3
-Text GLabel 7950 4650 2    60   Input ~ 0
+Text GLabel 7950 4450 2    60   Input ~ 0
 OUT_4
 Wire Wire Line
-	8000 2350 7900 2350
-Wire Wire Line
-	7950 4650 7850 4650
-Wire Wire Line
-	4950 4650 4850 4650
+	8000 2150 7900 2150
+Wire Wire Line
+	7950 4450 7850 4450
+Wire Wire Line
+	4950 4450 4850 4450
 Wire Wire Line
 	4950 2150 4850 2150
@@
 Connection ~ 6400 2250
 Wire Wire Line
-	4300 4650 4550 4650
-Wire Wire Line
 	4300 2350 4550 2350
-Wire Wire Line
-	7300 2350 7600 2350
-Wire Wire Line
-	7300 4650 7550 4650
 $Comp
 L MCP6V31U U1
@@
 F 3 "" H 4050 2450 50  0000 C CNN
 	1    4000 2250
-	-1   0    0    -1
+	-1   0    0    1
 $EndComp
 $Comp
@@
 Text Notes 4250 2700 0    60   ~ 0
 Put R3 in front of the + input.\nR3 = R1||R12
+$Comp
+L R R?
+U 1 1 5806BCB5
+P 4700 2350
+F 0 "R?" V 4780 2350 50  0000 C CNN
+F 1 "500K" V 4700 2350 50  0000 C CNN
+F 2 "Capacitors_SMD:C_0603" V 4630 2350 50  0001 C CNN
+F 3 "" H 4700 2350 50  0000 C CNN
+	1    4700 2350
+	0    1    1    0
+$EndComp
+Wire Wire Line
+	4850 2350 4950 2350
+$Comp
+L R R?
+U 1 1 5806BDA7
+P 7750 2350
+F 0 "R?" V 7830 2350 50  0000 C CNN
+F 1 "500K" V 7750 2350 50  0000 C CNN
+F 2 "Capacitors_SMD:C_0603" V 7680 2350 50  0001 C CNN
+F 3 "" H 7750 2350 50  0000 C CNN
+	1    7750 2350
+	0    1    1    0
+$EndComp
+$Comp
+L R R?
+U 1 1 5806BE58
+P 7700 4650
+F 0 "R?" V 7780 4650 50  0000 C CNN
+F 1 "500K" V 7700 4650 50  0000 C CNN
+F 2 "Capacitors_SMD:C_0603" V 7630 4650 50  0001 C CNN
+F 3 "" H 7700 4650 50  0000 C CNN
+	1    7700 4650
+	0    1    1    0
+$EndComp
+$Comp
+L R R?
+U 1 1 5806BEC4
+P 4700 4650
+F 0 "R?" V 4780 4650 50  0000 C CNN
+F 1 "500K" V 4700 4650 50  0000 C CNN
+F 2 "Capacitors_SMD:C_0603" V 4630 4650 50  0001 C CNN
+F 3 "" H 4700 4650 50  0000 C CNN
+	1    4700 4650
+	0    1    1    0
+$EndComp
+Wire Wire Line
+	7300 2150 7600 2150
+Wire Wire Line
+	7300 2350 7600 2350
+Wire Wire Line
+	7900 2350 8000 2350
+$Comp
+L MCP6V31U U?
+U 1 1 5806C5FA
+P 4000 4550
+F 0 "U?" H 4050 4750 50  0000 C CNN
+F 1 "MCP6V31U" H 4200 4350 50  0000 C CNN
+F 2 "" H 3950 4650 50  0000 C CNN
+F 3 "" H 4050 4750 50  0000 C CNN
+	1    4000 4550
+	-1   0    0    1
+$EndComp
+$Comp
+L MCP6V31U U?
+U 1 1 5806C651
+P 7000 4550
+F 0 "U?" H 7050 4750 50  0000 C CNN
+F 1 "MCP6V31U" H 7200 4350 50  0000 C CNN
+F 2 "" H 6950 4650 50  0000 C CNN
+F 3 "" H 7050 4750 50  0000 C CNN
+	1    7000 4550
+	-1   0    0    1
+$EndComp
+Wire Wire Line
+	4950 4650 4850 4650
+Wire Wire Line
+	4300 4450 4550 4450
+Wire Wire Line
+	4300 4650 4550 4650
+Wire Wire Line
+	7300 4450 7550 4450
+Wire Wire Line
+	7300 4650 7550 4650
+Wire Wire Line
+	7850 4650 8000 4650
 $EndSCHEMATC

Commit message: small changes
Parts:
- U26, U27: renamed from U?; footprint (none) -> TO_SOT_Packages_SMD:SC-70-5
- gave numbers to parts that had none: 4
Connections:
- net at R31.2, U27.3 (-): now also C44.1, R29.1
- net at R48.2, U27.1 (+): no longer C44.1, R29.1
Other:
- note removed: "470K = 0.102Hz\n680K = 0.07Hz\n1M = 0.048Hz\n2M = 0.024Hz\n3M3 = 0.015Hz"
- note removed: "Put R3 in front of the + input.\nR3 = R1||R12"
Changed lines of the file:
@@
 $Descr A4 11693 8268
 encoding utf-8
-Sheet 3 3
-Title ""
+Sheet 3 4
+Title "Ganglion Input Voltage References"
 Date ""
 Rev ""
-Comp ""
+Comp "OpenBCI, Inc"
 Comment1 ""
 Comment2 ""
@@
 V_REF
 $Comp
-L GNDA #PWR061
+L GNDA #PWR065
 U 1 1 57E27B47
 P 4100 2700
-F 0 "#PWR061" H 4100 2450 50  0001 C CNN
+F 0 "#PWR065" H 4100 2450 50  0001 C CNN
 F 1 "GNDA" H 4100 2550 50  0000 C CNN
 F 2 "" H 4100 2700 50  0000 C CNN
@@
 $EndComp
 $Comp
-L VAA #PWR062
+L VAA #PWR066
 U 1 1 57E27B67
 P 4100 1250
-F 0 "#PWR062" H 4100 1100 50  0001 C CNN
+F 0 "#PWR066" H 4100 1100 50  0001 C CNN
 F 1 "VAA" H 4100 1400 50  0000 C CNN
 F 2 "" H 4100 1250 50  0000 C CNN
@@
 Text Notes 2600 2000 0    60   ~ 0
 out to each ref
-Text Notes 3100 1400 0    60   ~ 0
-470K = 0.102Hz\n680K = 0.07Hz\n1M = 0.048Hz\n2M = 0.024Hz\n3M3 = 0.015Hz
 $Comp
 L C C37
@@
 $EndComp
 $Comp
-L GNDA #PWR063
+L GNDA #PWR067
 U 1 1 57EB84CB
 P 7100 2700
-F 0 "#PWR063" H 7100 2450 50  0001 C CNN
+F 0 "#PWR067" H 7100 2450 50  0001 C CNN
 F 1 "GNDA" H 7100 2550 50  0000 C CNN
 F 2 "" H 7100 2700 50  0000 C CNN
@@
 $EndComp
 $Comp
-L VAA #PWR064
+L VAA #PWR068
 U 1 1 57EB84EE
 P 7100 1300
-F 0 "#PWR064" H 7100 1150 50  0001 C CNN
+F 0 "#PWR068" H 7100 1150 50  0001 C CNN
 F 1 "VAA" H 7100 1450 50  0000 C CNN
 F 2 "" H 7100 1300 50  0000 C CNN
@@
 $EndComp
 $Comp
-L GNDA #PWR065
+L GNDA #PWR069
 U 1 1 57EB87DE
 P 4100 5100
-F 0 "#PWR065" H 4100 4850 50  0001 C CNN
+F 0 "#PWR069" H 4100 4850 50  0001 C CNN
 F 1 "GNDA" H 4100 4950 50  0000 C CNN
 F 2 "" H 4100 5100 50  0000 C CNN
@@
 $EndComp
 $Comp
-L GNDA #PWR066
+L GNDA #PWR070
 U 1 1 57EB8819
 P 7100 5100
-F 0 "#PWR066" H 7100 4850 50  0001 C CNN
+F 0 "#PWR070" H 7100 4850 50  0001 C CNN
 F 1 "GNDA" H 7100 4950 50  0000 C CNN
 F 2 "" H 7100 5100 50  0000 C CNN
@@
 $EndComp
 $Comp
-L VAA #PWR067
+L VAA #PWR071
 U 1 1 57EB8854
 P 7100 3600
-F 0 "#PWR067" H 7100 3450 50  0001 C CNN
+F 0 "#PWR071" H 7100 3450 50  0001 C CNN
 F 1 "VAA" H 7100 3750 50  0000 C CNN
 F 2 "" H 7100 3600 50  0000 C CNN
@@
 $EndComp
 $Comp
-L VAA #PWR068
+L VAA #PWR072
 U 1 1 57EB888F
 P 4100 3600
-F 0 "#PWR068" H 4100 3450 50  0001 C CNN
+F 0 "#PWR072" H 4100 3450 50  0001 C CNN
 F 1 "VAA" H 4100 3750 50  0000 C CNN
 F 2 "" H 4100 3600 50  0000 C CNN
@@
 Wire Wire Line
 	7000 3800 7450 3800
-Wire Wire Line
-	7450 3800 7450 4650
-Connection ~ 7450 4650
 Text GLabel 4950 2150 2    60   Input ~ 0
 OUT_1
@@
 	-1   0    0    1
 $EndComp
-Text Notes 4250 2700 0    60   ~ 0
-Put R3 in front of the + input.\nR3 = R1||R12
-$Comp
-L R R?
+$Comp
+L R R34
 U 1 1 5806BCB5
 P 4700 2350
-F 0 "R?" V 4780 2350 50  0000 C CNN
+F 0 "R34" V 4780 2350 50  0000 C CNN
 F 1 "500K" V 4700 2350 50  0000 C CNN
 F 2 "Capacitors_SMD:C_0603" V 4630 2350 50  0001 C CNN
@@
 	4850 2350 4950 2350
 $Comp
-L R R?
+L R R35
 U 1 1 5806BDA7
 P 7750 2350
-F 0 "R?" V 7830 2350 50  0000 C CNN
+F 0 "R35" V 7830 2350 50  0000 C CNN
 F 1 "500K" V 7750 2350 50  0000 C CNN
 F 2 "Capacitors_SMD:C_0603" V 7680 2350 50  0001 C CNN
@@
 $EndComp
 $Comp
-L R R?
+L R R48
 U 1 1 5806BE58
 P 7700 4650
-F 0 "R?" V 7780 4650 50  0000 C CNN
+F 0 "R48" V 7780 4650 50  0000 C CNN
 F 1 "500K" V 7700 4650 50  0000 C CNN
 F 2 "Capacitors_SMD:C_0603" V 7630 4650 50  0001 C CNN
@@
 $EndComp
 $Comp
-L R R?
+L R R36
 U 1 1 5806BEC4
 P 4700 4650
-F 0 "R?" V 4780 4650 50  0000 C CNN
+F 0 "R36" V 4780 4650 50  0000 C CNN
 F 1 "500K" V 4700 4650 50  0000 C CNN
 F 2 "Capacitors_SMD:C_0603" V 4630 4650 50  0001 C CNN
@@
 	7900 2350 8000 2350
 $Comp
-L MCP6V31U U?
+L MCP6V31U U26
 U 1 1 5806C5FA
 P 4000 4550
-F 0 "U?" H 4050 4750 50  0000 C CNN
+F 0 "U26" H 4050 4750 50  0000 C CNN
 F 1 "MCP6V31U" H 4200 4350 50  0000 C CNN
-F 2 "" H 3950 4650 50  0000 C CNN
+F 2 "TO_SOT_Packages_SMD:SC-70-5" H 3950 4650 50  0001 C CNN
 F 3 "" H 4050 4750 50  0000 C CNN
 	1    4000 4550
@@
 $EndComp
 $Comp
-L MCP6V31U U?
+L MCP6V31U U27
 U 1 1 5806C651
 P 7000 4550
-F 0 "U?" H 7050 4750 50  0000 C CNN
+F 0 "U27" H 7050 4750 50  0000 C CNN
 F 1 "MCP6V31U" H 7200 4350 50  0000 C CNN
-F 2 "" H 6950 4650 50  0000 C CNN
+F 2 "TO_SOT_Packages_SMD:SC-70-5" H 6950 4650 50  0001 C CNN
 F 3 "" H 7050 4750 50  0000 C CNN
 	1    7000 4550
@@
 Wire Wire Line
 	7850 4650 8000 4650
+Wire Wire Line
+	7450 3800 7450 4450
+Connection ~ 7450 4450
 $EndSCHEMATC
