File: Ganglion_KiCad_Files/References.sch (KiCad schematic (older format))
At the start: 20 parts, among them U1 MCP6V31U, U24 MCP6V31U, U26 MCP6V31U, U27 MCP6V31U

Commit message: Annotate components with manufacturer part numbers
Parts:
- C37, C39, C44, C9: ManufacturerPartNumber (none) -> GRM188R60J226MEA0D
- R1, R10, R12, R13, R14, R29, R30, R31: ManufacturerPartNumber (none) -> ERJ-3EKF1004V
- R34, R35, R36, R48: ManufacturerPartNumber (none) -> CR0603-FX-4993ELF
- U1, U24, U26, U27: ManufacturerPartNumber (none) -> MCP6V31UT-E/LT
Changed lines of the file:
@@
 F 2 "Capacitors_SMD:C_0603" H 3888 1650 50  0001 C CNN
 F 3 "" H 3850 1800 50  0000 C CNN
+F 4 "GRM188R60J226MEA0D" V 3850 1800 60  0001 C CNN "ManufacturerPartNumber"
 	1    3850 1800
 	0    1    1    0
@@
 F 2 "Capacitors_SMD:C_0603" V 3780 1500 50  0001 C CNN
 F 3 "" H 3850 1500 50  0000 C CNN
+F 4 "ERJ-3EKF1004V" H 3850 1500 60  0001 C CNN "ManufacturerPartNumber"
 	1    3850 1500
 	0    1    1    0
@@
 F 2 "Capacitors_SMD:C_0603" V 4630 2350 50  0001 C CNN
 F 3 "" H 4700 2350 50  0000 C CNN
+F 4 "ERJ-3EKF1004V" H 4700 2350 60  0001 C CNN "ManufacturerPartNumber"
 	1    4700 2350
 	0    1    1    0
@@
 F 2 "Capacitors_SMD:C_0603" H 6888 1650 50  0001 C CNN
 F 3 "" H 6850 1800 50  0000 C CNN
+F 4 "GRM188R60J226MEA0D" V 6850 1800 60  0001 C CNN "ManufacturerPartNumber"
 	1    6850 1800
 	0    1    1    0
@@
 F 2 "Capacitors_SMD:C_0603" V 6780 1500 50  0001 C CNN
 F 3 "" H 6850 1500 50  0000 C CNN
+F 4 "ERJ-3EKF1004V" H 6850 1500 60  0001 C CNN "ManufacturerPartNumber"
 	1    6850 1500
 	0    1    1    0
@@
 F 2 "Capacitors_SMD:C_0603" V 7680 2350 50  0001 C CNN
 F 3 "" H 7750 2350 50  0000 C CNN
+F 4 "ERJ-3EKF1004V" H 7750 2350 60  0001 C CNN "ManufacturerPartNumber"
 	1    7750 2350
 	0    1    1    0
@@
 F 2 "Capacitors_SMD:C_0603" H 3888 3950 50  0001 C CNN
 F 3 "" H 3850 4100 50  0000 C CNN
+F 4 "GRM188R60J226MEA0D" V 3850 4100 60  0001 C CNN "ManufacturerPartNumber"
 	1    3850 4100
 	0    1    1    0
@@
 F 2 "Capacitors_SMD:C_0603" V 3780 3800 50  0001 C CNN
 F 3 "" H 3850 3800 50  0000 C CNN
+F 4 "ERJ-3EKF1004V" H 3850 3800 60  0001 C CNN "ManufacturerPartNumber"
 	1    3850 3800
 	0    1    1    0
@@
 F 2 "Capacitors_SMD:C_0603" V 4630 4650 50  0001 C CNN
 F 3 "" H 4700 4650 50  0000 C CNN
+F 4 "ERJ-3EKF1004V" H 4700 4650 60  0001 C CNN "ManufacturerPartNumber"
 	1    4700 4650
 	0    1    1    0
@@
 F 2 "Capacitors_SMD:C_0603" V 7630 4650 50  0001 C CNN
 F 3 "" H 7700 4650 50  0000 C CNN
+F 4 "ERJ-3EKF1004V" H 7700 4650 60  0001 C CNN "ManufacturerPartNumber"
 	1    7700 4650
 	0    1    1    0
@@
 F 2 "Capacitors_SMD:C_0603" H 6888 3950 50  0001 C CNN
 F 3 "" H 6850 4100 50  0000 C CNN
+F 4 "GRM188R60J226MEA0D" V 6850 4100 60  0001 C CNN "ManufacturerPartNumber"
 	1    6850 4100
 	0    1    1    0
@@
 F 2 "Capacitors_SMD:C_0603" V 6780 3800 50  0001 C CNN
 F 3 "" H 6850 3800 50  0000 C CNN
+F 4 "ERJ-3EKF1004V" H 6850 3800 60  0001 C CNN "ManufacturerPartNumber"
 	1    6850 3800
 	0    1    1    0
@@
 F 2 "TO_SOT_Packages_SMD:SC-70-5" H 3950 2350 50  0001 C CNN
 F 3 "" H 4050 2450 50  0000 C CNN
+F 4 "MCP6V31UT-E/LT" H 4000 2250 60  0001 C CNN "ManufacturerPartNumber"
 	1    4000 2250
 	-1   0    0    -1
@@
 F 2 "TO_SOT_Packages_SMD:SC-70-5" H 6950 2350 50  0001 C CNN
 F 3 "" H 7050 2450 50  0000 C CNN
+F 4 "MCP6V31UT-E/LT" H 7000 2250 60  0001 C CNN "ManufacturerPartNumber"
 	1    7000 2250
 	-1   0    0    -1
@@
 F 2 "Capacitors_SMD:C_0603" V 4630 2150 50  0001 C CNN
 F 3 "" H 4700 2150 50  0000 C CNN
+F 4 "CR0603-FX-4993ELF" V 4700 2150 60  0001 C CNN "ManufacturerPartNumber"
 	1    4700 2150
 	0    1    1    0
@@
 F 2 "Capacitors_SMD:C_0603" V 7680 2150 50  0001 C CNN
 F 3 "" H 7750 2150 50  0000 C CNN
+F 4 "CR0603-FX-4993ELF" V 7750 2150 60  0001 C CNN "ManufacturerPartNumber"
 	1    7750 2150
 	0    1    1    0
@@
 F 2 "Capacitors_SMD:C_0603" V 7630 4450 50  0001 C CNN
 F 3 "" H 7700 4450 50  0000 C CNN
+F 4 "CR0603-FX-4993ELF" V 7700 4450 60  0001 C CNN "ManufacturerPartNumber"
 	1    7700 4450
 	0    1    1    0
@@
 F 2 "Capacitors_SMD:C_0603" V 4630 4450 50  0001 C CNN
 F 3 "" H 4700 4450 50  0000 C CNN
+F 4 "CR0603-FX-4993ELF" V 4700 4450 60  0001 C CNN "ManufacturerPartNumber"
 	1    4700 4450
 	0    1    1    0
@@
 F 2 "TO_SOT_Packages_SMD:SC-70-5" H 3950 4650 50  0001 C CNN
 F 3 "" H 4050 4750 50  0000 C CNN
+F 4 "MCP6V31UT-E/LT" H 4000 4550 60  0001 C CNN "ManufacturerPartNumber"
 	1    4000 4550
 	-1   0    0    -1
@@
 F 2 "TO_SOT_Packages_SMD:SC-70-5" H 6950 4650 50  0001 C CNN
 F 3 "" H 7050 4750 50  0000 C CNN
+F 4 "MCP6V31UT-E/LT" H 7000 4550 60  0001 C CNN "ManufacturerPartNumber"
 	1    7000 4550
 	-1   0    0    -1
