File: Ganglion_KiCad_Files/TVS.sch (KiCad schematic (older format))
At the start: 3 parts, among them U28 TPD4E1B06, U29 TPD4E1B06, U30 TPD4E1B06

Commit message: Annotate components with manufacturer part numbers
Parts:
- U28, U29, U30: ManufacturerPartNumber (none) -> TPD4E1B06DCKR
Changed lines of the file:
@@
 F 2 "TO_SOT_Packages_SMD:SC-70-6" H 3100 1400 60  0001 C CNN
 F 3 "" H 3100 1400 60  0000 C CNN
+F 4 "TPD4E1B06DCKR" H 3100 1400 60  0001 C CNN "ManufacturerPartNumber"
 	1    3100 1400
 	1    0    0    -1
@@
 F 2 "TO_SOT_Packages_SMD:SC-70-6" H 3100 2350 60  0001 C CNN
 F 3 "" H 3100 2350 60  0000 C CNN
+F 4 "TPD4E1B06DCKR" H 3100 2350 60  0001 C CNN "ManufacturerPartNumber"
 	1    3100 2350
 	1    0    0    -1
@@
 F 2 "TO_SOT_Packages_SMD:SC-70-6" H 4900 1400 60  0001 C CNN
 F 3 "" H 4900 1400 60  0000 C CNN
+F 4 "TPD4E1B06DCKR" H 4900 1400 60  0001 C CNN "ManufacturerPartNumber"
 	1    4900 1400
 	1    0    0    -1
