File: Ganglion_KiCad_Files/Ganglion_01.kicad_pcb (KiCad board)
At the start: 4 copper layers, 61.2 x 61.2 mm, 141 parts, among them P1 CONN_02X08, P2 CONN_01X04, P3 CONN_01X04, P4 CONN_01X08, P5 CONN_01X08, SW1 CJS1200, SW2 CJS1200, SW3 CJS1200, SW4 CJS1200, SW5 SPDT, SW6 TACT_SWITCH, U1 MCP6V31U, U10 NCP300, U11 NCP551, U12 AD5621, U13 SEEED_microSD, U14 MCP6V13T, U15 MCP6001, U16 SN74LVC1G32, U17 LIS2DE12, U18 74LVC1G66, U19 74LVC1G66, U2 AD8237, U20 74LVC1G66, U21 74LVC1G66, U22 74LVC1G66, U23 74LVC2G00, U24 MCP6V31U, U25 MCP6V31U, U26 MCP6V31U, U27 MCP6V31U, U28 TPD4E1B06, U29 TPD4E1B06, U3 AD8237, U30 TPD4E1B06, U4 AD8237, U5 AD8237, U6 LM7332, U7 MCP3912, U8 rfd_77101, U9 NCP551, Y1 Crystal_Small

Commit message: Fix discrepancies between schematic/board values and the BOM
Parts:
- C35: value 100uF -> 47uF
- C37, C39, C44, C9: value 3.3uF -> 22uF
- R49: value 470K -> 330K
Changed lines of the file:
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@@
       (effects (font (size 0.75 0.75) (thickness 0.15)) (justify mirror))
     )
-    (fp_text value 3.3uF (at 0 -1.9) (layer B.Fab)
+    (fp_text value 22uF (at 0 -1.9) (layer B.Fab)
       (effects (font (size 1 1) (thickness 0.15)) (justify mirror))
     )
@@
       (effects (font (size 0.75 0.75) (thickness 0.15)) (justify mirror))
     )
-    (fp_text value 100uF (at 0 -2.7 135) (layer B.Fab)
+    (fp_text value 47uF (at 0 -2.7 135) (layer B.Fab)
       (effects (font (size 1 1) (thickness 0.15)) (justify mirror))
     )
@@
       (effects (font (size 0.75 0.75) (thickness 0.15)) (justify mirror))
     )
-    (fp_text value 3.3uF (at 0 -1.9) (layer B.Fab)
+    (fp_text value 22uF (at 0 -1.9) (layer B.Fab)
       (effects (font (size 1 1) (thickness 0.15)) (justify mirror))
     )
@@
       (effects (font (size 0.75 0.75) (thickness 0.15)) (justify mirror))
     )
-    (fp_text value 3.3uF (at 0 -1.9) (layer B.Fab)
+    (fp_text value 22uF (at 0 -1.9) (layer B.Fab)
       (effects (font (size 1 1) (thickness 0.15)) (justify mirror))
     )
@@
       (effects (font (size 0.75 0.75) (thickness 0.15)) (justify mirror))
     )
-    (fp_text value 3.3uF (at 0 -1.9) (layer B.Fab)
+    (fp_text value 22uF (at 0 -1.9) (layer B.Fab)
       (effects (font (size 1 1) (thickness 0.15)) (justify mirror))
     )
@@
       (effects (font (size 0.75 0.75) (thickness 0.15)))
     )
-    (fp_text value 470K (at 0 1.9) (layer F.Fab)
+    (fp_text value 330K (at 0 1.9) (layer F.Fab)
       (effects (font (size 1 1) (thickness 0.15)))
     )
